File: pcb/attiny85_remote.kicad_pcb (KiCad board)
At the start: 2 copper layers, 24.2 x 70 mm, 37 parts, among them J3 RST/PWR, J4 Conn_01x02_Pin, J5 PWR, J6 Conn_01x02_Pin, J7 Conn_01x02_Pin, Q2 AO3401A, SW1 F2, SW2 F2, SW3 F2, U1 Ai-Thinker-Ra-02, t85 ATTINY85-20MU

Commit message: rework done
Parts:
- removed ?: , 
- removed D2: D, Diode_THT:D_DO-35_SOD27_P7.62mm_Horizontal
- removed J4, J6, J7: Conn_01x02_Pin, Jumper:SolderJumper-2_P1.3mm_Open_Pad1.0x1.5mm
- removed J5: PWR, Jumper:SolderJumper-2_P1.3mm_Open_Pad1.0x1.5mm
- removed the REF** at (201.7, 49.6)
- removed the REF** at (196.0, 46.2)
- removed the REF** at (188.2, 49.9)
- removed the REF** at (186.0, 96.0)
- removed the REF** at (197.2, 58.7)
- removed the REF** at (195.1, 55.9)
- removed the REF** at (192.8, 46.1)
- removed the REF** at (189.4, 95.9)
- removed the REF** at (180.4, 49.7)
- removed the REF** at (193.7, 83.3)
- removed the REF** at (193.5, 63.8)
- removed the REF** at (180.4, 60.2)
- removed the REF** at (201.7, 60.2)
- removed the REF** at (189.6, 46.1)
- removed the REF** at (193.4, 96.0)
- removed the REF** at (186.1, 46.1)
- removed t85: ATTINY85-20MU, Custom:QFN50P400X400X80-21N-D
- added D6: D, Diode_THT:D_DO-35_SOD27_P7.62mm_Horizontal, B.Cu at (201.6, 54.3)
- added IC1: ATTINY85-20MU, Custom:QFN50P400X400X80-21N-D, B.Cu at (191.1, 54.9)
- added J1: RST/DRV, Jumper:SolderJumper-3_P1.3mm_Open_Pad1.0x1.5mm, B.Cu at (188.0, 60.4)
- added J2: INT/DRV, Jumper:SolderJumper-3_P1.3mm_Open_Pad1.0x1.5mm, B.Cu at (194.5, 60.4)
- added REF**: SolderWirePad_1x01_SMD_1x2mm, Connector_Wire:SolderWirePad_1x01_SMD_1x2mm, B.Cu at (187.8, 46.5)
- added REF**: SolderWirePad_1x01_SMD_1x2mm, Connector_Wire:SolderWirePad_1x01_SMD_1x2mm, B.Cu at (194.4, 46.5)
- added REF**: SolderWirePad_1x01_SMD_1x2mm, Connector_Wire:SolderWirePad_1x01_SMD_1x2mm, B.Cu at (185.6, 46.5)
- added REF**: SolderWirePad_1x01_SMD_1x2mm, Connector_Wire:SolderWirePad_1x01_SMD_1x2mm, B.Cu at (190.0, 46.5)
- added REF**: SolderWirePad_1x01_SMD_1x2mm, Connector_Wire:SolderWirePad_1x01_SMD_1x2mm, B.Cu at (193.9, 96.3)
- added REF**: SolderWirePad_1x01_SMD_1x2mm, Connector_Wire:SolderWirePad_1x01_SMD_1x2mm, B.Cu at (196.6, 46.5)
- added REF**: SolderWirePad_1x01_SMD_1x2mm, Connector_Wire:SolderWirePad_1x01_SMD_1x2mm, B.Cu at (188.2, 96.3)
- added REF**: SolderWirePad_1x01_SMD_1x2mm, Connector_Wire:SolderWirePad_1x01_SMD_1x2mm, B.Cu at (192.2, 46.5)
- C1, C2: value 100uF -> 1000uF
- J3: value RST/PWR -> PWR; footprint Jumper:SolderJumper-3_P1.3mm_Open_Pad1.0x1.5mm -> Jumper:SolderJumper-2_P1.3mm_Open_Pad1.0x1.5mm
- moved D5 14.2 mm to (201.6, 56.4), turned to -90 degrees
- moved D1 10.4 mm to (194.9, 63.8), turned to 180 degrees
- moved SW2 8.25 mm to (180.6, 66.5)
- moved SW3 8.25 mm to (188.8, 66.5)
- moved SW1 7.91 mm to (201.6, 73.0), turned to 90 degrees
- moved Q2 3.64 mm to (189.6, 80.6), turned to -90 degrees
- moved J3 2.63 mm to (189.2, 85.0), turned to 180 degrees
- moved R1 0.94 mm to (193.1, 76.5)
- moved D3 0.40 mm to (180.6, 56.4)
- moved D4 0.40 mm to (180.6, 54.3)
Connections:
- D1 pad 1: /INT0 -> Net-(D1-K)
- D3 pad 1: /INT0 -> Net-(D1-K)
- D3 pad 2: /PB1_SW -> Net-(D3-A)
- D4 pad 2: /PB1_SW -> Net-(D3-A)
- D5 pad 1: /INT0 -> Net-(D1-K)
- J3 pad 1: /RST -> +3.3V
- J3 pad 2: /PB4 -> VCC
- Q2 pad 1: /CLAMP -> /DRV
- R1 pad 2: /CLAMP -> /DRV
- SW2 pad 1: /SW2 -> Net-(D3-A)
Routing:
- net Net-(D1-A): track 54.8 -> 9.90 mm
- net /INT0: track 63.3 -> 20.2 mm, vias 4 -> 3
- net /CLAMP: track 34.5 -> 0.00 mm, vias 3 -> 0
- net /PB1_SW: track 33.2 -> 0.00 mm
- net /DRV: track 0.00 -> 31.8 mm, vias 0 -> 1
- net Net-(D1-K): track 0.00 -> 31.2 mm
- net /RST: track 39.8 -> 9.01 mm, vias 2 -> 1
- net /MISO: track 54.5 -> 24.8 mm, vias 2 -> 5
- net Net-(D3-A): track 0.00 -> 27.3 mm
- net /PB3: track 50.5 -> 24.6 mm, vias 3 -> 2
- net /SW2: track 20.5 -> 0.00 mm
- net /MOSI: track 41.3 -> 21.3 mm
- net Net-(D5-A): track 11.6 -> 27.4 mm, vias 1 -> 0
- net +3.3V: track 52.8 -> 43.5 mm, vias 5 -> 1
- net /PB5: track 30.4 -> 21.7 mm, vias 3 -> 2
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Other:
- board text removed: "PB0"
- board text removed: "PB1"
- board text removed: "PB2"
- board text removed: "PB3"

Commit message: gerber out
Parts:
- removed Q2: AO3401A, Package_TO_SOT_SMD:SOT-23
- added Q1: SSM3J35AFS,LF, Custom:SSM3J35AFSLF, F.Cu at (192.5, 82.3)
- added R2: 100, Resistor_THT:R_Axial_DIN0207_L6.3mm_D2.5mm_P10.16mm_Horizontal, B.Cu at (188.9, 85.8)
- added REF**: SolderWirePad_1x01_SMD_1x2mm, Connector_Wire:SolderWirePad_1x01_SMD_1x2mm, B.Cu at (195.4, 53.9)
- R1: value 10k -> 22k; moved to B.Cu
- U1: value Ai-Thinker-Ra-02 -> Ra-02
- moved J3 9.53 mm to (192.7, 76.2)
- moved D4 7.62 mm to (180.6, 46.7), turned to -90 degrees
- moved D3 7.61 mm to (180.6, 64.0), turned to 90 degrees
- moved D5 7.61 mm to (201.6, 64.0), turned to 90 degrees
- moved D6 7.61 mm to (201.6, 46.7), turned to -90 degrees
- moved D1 7.61 mm to (187.3, 63.8), turned to 0 degrees
- moved C2 4.98 mm to (185.7, 90.5), turned to 180 degrees
- moved R1 1.91 mm to (193.3, 78.4)
- renumbered IC1 to Attiny85
Connections:
- D3 pad 1: Net-(D1-K) -> Net-(D3-K)
- D3 pad 2: Net-(D3-A) -> Net-(D1-A)
- D4 pad 1: /MISO -> Net-(D3-K)
- D4 pad 2: Net-(D3-A) -> /MISO
- D5 pad 1: Net-(D1-K) -> Net-(D5-K)
- D5 pad 2: Net-(D5-A) -> Net-(D1-A)
- D6 pad 1: /MOSI -> Net-(D5-K)
- D6 pad 2: Net-(D5-A) -> /MOSI
- J2 pad 2: Net-(D1-K) -> Net-(D1-A)
- R1 pad 2: /DRV -> Net-(Q1-G)
- SW1 pad 1: Net-(D5-A) -> Net-(D5-K)
- SW2 pad 1: Net-(D3-A) -> Net-(D3-K)
- SW3 pad 1: Net-(D1-A) -> Net-(D1-K)
Routing:
- net Net-(D5-K): track 0.00 -> 27.4 mm
- net Net-(D5-A): track 27.4 -> 0.00 mm
- net Net-(D3-A): track 27.3 -> 0.00 mm
- net Net-(D3-K): track 0.00 -> 27.3 mm
- net Net-(D1-A): track 9.90 -> 31.2 mm
- net Net-(D1-K): track 31.2 -> 9.90 mm
- net Net-(Q1-G): track 0.00 -> 12.2 mm
- net /DRV: track 31.8 -> 19.9 mm
- net +3.3V: track 43.5 -> 46.6 mm, vias 1 -> 0
- net VCC: track 45.2 -> 43.8 mm
- net GND: vias 35 -> 37
Other:
- board text added: "DRV"
- board text added: "INT"
- board text added: "PB0"
- board text added: "PB1"
- board text added: "PB2"
- board text added: "PB3"
- board text removed: "BTN"
- board text removed: "CL"
- board text removed: "PWR"
