File: pcb/attiny85_remote.kicad_sch (KiCad schematic)
At the start: 22 parts, among them IC1 ATTINY85-20MU, J1 GPIO, J2 PWR, J3 RST/PWR, J4 Conn_01x02_Pin, J5 PWR, J6 Conn_01x02_Pin, J7 Conn_01x02_Pin, Q2 AO3401A, SW1 F2, SW2 F2, SW3 F2, U1 Ai-Thinker-Ra-02

Commit message: before rework
Parts:
- removed D2: D, Diode_THT:D_DO-35_SOD27_P7.62mm_Horizontal, symbol Device:D_Small
- removed J1: GPIO, Connector_PinHeader_2.54mm:PinHeader_1x06_P2.54mm_Horizontal, symbol Connector:Conn_01x06_Pin
- removed J2: PWR, Connector_PinHeader_2.54mm:PinHeader_1x02_P2.54mm_Horizontal, symbol Connector:Conn_01x02_Pin
- removed J3: RST/PWR, Jumper:SolderJumper-3_P1.3mm_Open_Pad1.0x1.5mm, symbol Connector:Conn_01x03_Pin
- removed J4, J6, J7: Conn_01x02_Pin, Jumper:SolderJumper-2_P1.3mm_Open_Pad1.0x1.5mm, symbol Connector:Conn_01x02_Pin
- removed J5: PWR, Jumper:SolderJumper-2_P1.3mm_Open_Pad1.0x1.5mm, symbol Connector:Conn_01x02_Pin
- added D6: D, Diode_THT:D_DO-35_SOD27_P7.62mm_Horizontal, symbol Device:D_Small
- added J1: RST/DRV, Jumper:SolderJumper-3_P1.3mm_Open_Pad1.0x1.5mm, symbol Connector:Conn_01x03_Pin
- added J2: INT/DRV, symbol Connector:Conn_01x03_Pin
- C1, C2: value 100uF -> 1000uF
Connections:
- net SW2 is gone; now on an unnamed net: SW2.1
- net INT0: now also J2.3 (Pin_3); no longer D1.1 (K), D3.1 (K), D5.1 (K)
- net MOSI: now also D6.1 (K)
- net PB4: now also J1.2 (Pin_2)
- net RST: now also J1.1 (Pin_1)
- net at D5.2 (A), SW1.1: now also D6.2 (A)
- net CLAMP renamed DRV
- net DRV: now also J1.3 (Pin_3), J2.1 (Pin_1)
- net PB1_SW: no longer names the net of D3.2 (A), D4.2 (A)
- new net: D1.1 (K), D3.1 (K), D5.1 (K), J2.2 (Pin_2)
Other:
- note added: "TODO: LoRa Reset pullup?"
- moved on the sheet: BT1, C1, C2, D1, D3, D4, Q2, R1, SW1, SW2, SW3

Commit message: rework done
Parts:
- added J3: PWR, Jumper:SolderJumper-2_P1.3mm_Open_Pad1.0x1.5mm, symbol Connector:Conn_01x02_Pin
- J2: footprint (none) -> Jumper:SolderJumper-3_P1.3mm_Open_Pad1.0x1.5mm
Connections:
- net +3.3V: now also J3.1 (Pin_1)
- net DRV: now also J1.1 (Pin_1); no longer J1.3 (Pin_3)
- net RST: now also J1.3 (Pin_3); no longer J1.1 (Pin_1)
- net VCC: now also J3.2 (Pin_2)
Other:
- note removed: "TODO: LoRa Reset pullup?"
Changed lines of the file:
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@@
+    (stroke (width 0) (type default))
+  )
+  (wire (pts (xy 191.77 44.45) (xy 196.85 44.45))
+    (stroke (width 0) (type default))
+  )
+  (wire (pts (xy 91.44 95.25) (xy 96.52 95.25))
+    (stroke (width 0) (type default))
+  )
+  (wire (pts (xy 63.5 114.3) (xy 63.5 115.57))
     (stroke (width 0) (type default))
   )
@@
     (stroke (width 0) (type default))
   )
-  (wire (pts (xy 191.77 44.45) (xy 196.85 44.45))
-    (stroke (width 0) (type default))
-  )
-  (wire (pts (xy 91.44 95.25) (xy 96.52 95.25))
-    (stroke (width 0) (type default))
-  )
-  (wire (pts (xy 63.5 114.3) (xy 63.5 115.57))
-    (stroke (width 0) (type default))
-  )
   (wire (pts (xy 43.18 105.41) (xy 48.26 105.41))
     (stroke (width 0) (type default))
@@
     (stroke (width 0) (type default))
   )
-  (text "TODO: LoRa Reset pullup?" (at 102.87 92.71 0)
-    (effects (font (size 1.27 1.27)) (justify left bottom))
-  )
   (label "PB0" (at 82.55 55.88 180) (fields_autoplaced)
     (effects (font (size 1.27 1.27)) (justify right bottom))
@@
     (effects (font (size 1.27 1.27)) (justify right bottom))
   )
-  (label "DRV" (at 96.52 97.79 180) (fields_autoplaced)
+  (label "DRV" (at 96.52 92.71 180) (fields_autoplaced)
     (effects (font (size 1.27 1.27)) (justify right bottom))
   )
@@
     (effects (font (size 1.27 1.27)) (justify left bottom))
   )
-  (label "RST" (at 96.52 92.71 180) (fields_autoplaced)
+  (label "RST" (at 96.52 97.79 180) (fields_autoplaced)
     (effects (font (size 1.27 1.27)) (justify right bottom))
   )
@@
     )
   )
+  (symbol (lib_id "Connector:Conn_01x02_Pin") (at 165.1 64.77 0) (unit 1)
+    (in_bom yes) (on_board yes) (dnp no) (fields_autoplaced)
+    (property "Reference" "J3" (at 165.735 60.96 0)
+      (effects (font (size 1.27 1.27)))
+    )
+    (property "Value" "PWR" (at 165.735 63.5 0)
+      (effects (font (size 1.27 1.27)))
+    )
+    (property "Footprint" "Jumper:SolderJumper-2_P1.3mm_Open_Pad1.0x1.5mm" (at 165.1 64.77 0)
+      (effects (font (size 1.27 1.27)) hide)
+    )
+    (property "Datasheet" "~" (at 165.1 64.77 0)
+      (effects (font (size 1.27 1.27)) hide)
+    )
+    (pin "1")
+    (pin "2")
+    (instances
+      (project "attiny85_remote"
+        (path "/db7d5605-f896-494c-b27c-eb6bf0dfb607"
+          (reference "J3") (unit 1)
+        )
+      )
+    )
+  )
   (symbol (lib_id "Device:D_Small") (at 50.8 100.33 0) (unit 1)
     (in_bom yes) (on_board yes) (dnp no)
@@
   )
   (symbol (lib_id "Connector:Conn_01x03_Pin") (at 24.13 100.33 0) (unit 1)
-    (in_bom yes) (on_board yes) (dnp no) (fields_autoplaced)
+    (in_bom yes) (on_board yes) (dnp no)
     (property "Reference" "J2" (at 24.765 93.98 0)
       (effects (font (size 1.27 1.27)))
@@
       (effects (font (size 1.27 1.27)))
     )
-    (property "Footprint" "" (at 24.13 100.33 0)
+    (property "Footprint" "Jumper:SolderJumper-3_P1.3mm_Open_Pad1.0x1.5mm" (at 24.13 100.33 0)
       (effects (font (size 1.27 1.27)) hide)
     )
@@
     )
   )
+  (symbol (lib_id "power:+3.3V") (at 170.18 64.77 0) (unit 1)
+    (in_bom yes) (on_board yes) (dnp no) (fields_autoplaced)
+    (property "Reference" "#PWR04" (at 170.18 68.58 0)
+      (effects (font (size 1.27 1.27)) hide)
+    )
+    (property "Value" "+3.3V" (at 170.18 60.96 0)
+      (effects (font (size 1.27 1.27)))
+    )
+    (property "Footprint" "" (at 170.18 64.77 0)
+      (effects (font (size 1.27 1.27)) hide)
+    )
+    (property "Datasheet" "" (at 170.18 64.77 0)
+      (effects (font (size 1.27 1.27)) hide)
+    )
+    (pin "1")
+    (instances
+      (project "attiny85_remote"
+        (path "/db7d5605-f896-494c-b27c-eb6bf0dfb607"
+          (reference "#PWR04") (unit 1)
+        )
+      )
+    )
+  )
   (symbol (lib_id "Device:D_Small") (at 50.8 111.76 0) (unit 1)
     (in_bom yes) (on_board yes) (dnp no)
@@
         )
       )
+    )
+  )
+  (symbol (lib_id "power:VCC") (at 170.18 67.31 180) (unit 1)
+    (in_bom yes) (on_board yes) (dnp no) (fields_autoplaced)
+    (property "Reference" "#PWR01" (at 170.18 63.5 0)
+      (effects (font (size 1.27 1.27)) hide)
+    )
+    (property "Value" "VCC" (at 170.18 72.39 0)
+      (effects (font (size 1.27 1.27)))
+    )
+    (property "Footprint" "" (at 170.18 67.31 0)
+      (effects (font (size 1.27 1.27)) hide)
+    )
+    (property "Datasheet" "" (at 170.18 67.31 0)
+      (effects (font (size 1.27 1.27)) hide)
+    )
+    (pin "1")
+    (instances
+      (project "attiny85_remote"
+        (path "/db7d5605-f896-494c-b27c-eb6bf0dfb607"
+          (reference "#PWR01") (unit 1)
+        )
+      )

Commit message: gerber out
Parts:
- removed Q2: AO3401A, Package_TO_SOT_SMD:SOT-23, symbol Transistor_FET:AO3401A
- added Q1: SSM3J35AFS,LF, Custom:SSM3J35AFSLF, symbol Custom:SSM3J35AFS,LF
- added R2: 100, Resistor_THT:R_Axial_DIN0207_L6.3mm_D2.5mm_P10.16mm_Horizontal, symbol Device:R_Small
- R1: value 10k -> 22k
Connections:
- net +3.3V: now also Q1.2 (S)
- net DRV: now also R2.2; no longer R1.2
- net MISO: now also D4.2 (A); no longer D4.1 (K)
- net MOSI: now also D6.2 (A); no longer D6.1 (K)
- net VCC: now also Q1.3 (D)
- net at SW3.1: now also D1.1 (K); no longer D1.2 (A)
- new net: D1.2 (A), D3.2 (A), D5.2 (A), J2.2 (Pin_2)
- new net: Q1.1 (G), R1.2, R2.1
- new net: D3.1 (K), D4.1 (K), SW2.1
- new net: D5.1 (K), D6.1 (K), SW1.1
Other:
- moved on the sheet: BT1, C1, C2, D1, D3, D4, D5, D6, J1, J2, J3, R1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
