File: pcb/attiny1624_remote.kicad_sch (KiCad schematic)
At the start: 25 parts, among them J4 UPDI, J5 UART0, Q1 BSS138, SW1 F2, SW2 F2, SW3 F2, U1 DL-LLCC68-S-433, U2 ATtiny1624-X, U3 VG433SNX39-6W3

Commit message: pcb done?
Parts:
- added J1: JMP, Connector_PinHeader_2.54mm:PinHeader_1x02_P2.54mm_Vertical, symbol Connector_Generic:Conn_01x02
Connections:
- net VCC is gone; now on net +3.3V: J4.2 (Pin_2), SW1.2, SW2.2, SW3.2, U1.3 (3.3V), U2.1 (VCC)
- net +3.3V: now also J1.1 (Pin_1)
- net BTN1: now also D1.2 (A)
- net BTN2: now also D2.2 (A), U2.3 (PA5); no longer U2.5 (PA7)
- net GND: no longer U1.16 (GND), U1.2 (GND), U1.9 (GND)
- net NMOS: now also U1.16 (GND), U1.2 (GND), U1.9 (GND)
- net RST: now also U2.5 (PA7); no longer U2.3 (PA5)
- net STRAP: now also J1.2 (Pin_2)
