File: pcb/attiny1624_remote.kicad_pcb (KiCad board)
At the start: 2 copper layers, 30 x 70 mm, 26 parts, among them J4 UPDI, J5 UART0, Q1 BSS138, SW1 F2, SW2 F2, SW3 F2, U1 DL-LLCC68-S-433, U2 ATtiny1624-X, U3 VG433SNX39-6W3

Commit message: pcb done?
Parts:
- added J1: JMP, Connector_PinHeader_2.54mm:PinHeader_1x02_P2.54mm_Vertical, F.Cu at (114.8, 74.0)
- BT1, C1, C2: moved to F.Cu
- G***: moved to B.Cu
- moved J4 66.9 mm to (112.2, 76.6), turned to 90 degrees
- moved C5 57.3 mm to (99.2, 48.6), turned to -90 degrees
- moved R3 53.0 mm to (112.4, 67.5), turned to -90 degrees
- moved C6 44.3 mm to (99.3, 45.0), turned to 90 degrees
- moved D2 40.3 mm to (114.3, 67.8), turned to 90 degrees
- moved C3 40.1 mm to (125.3, 55.1), turned to -90 degrees
- moved C4 37.2 mm to (126.9, 55.1), turned to -90 degrees
- moved R1 34.2 mm to (117.2, 71.0), turned to 0 degrees
- moved R5 32.4 mm to (121.8, 41.3), turned to 90 degrees
- moved J5 28.9 mm to (125.4, 46.0), turned to -90 degrees
- moved R4 27.9 mm to (126.5, 41.3), turned to 90 degrees
- moved D1 26.8 mm to (110.5, 67.9), turned to 90 degrees
- moved Q1 19.6 mm to (117.2, 68.1)
- moved D4 16.9 mm to (125.0, 41.3), turned to 90 degrees
- moved R2 16.7 mm to (108.7, 67.5), turned to -90 degrees
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Connections:
- D1 pad 2: Net-(D1-A) -> /BTN1
- D2 pad 2: Net-(D2-A) -> /BTN2
- J4 pad 2: VCC -> +3.3V
- SW1 pad 2: VCC -> +3.3V
- SW2 pad 2: VCC -> +3.3V
- SW3 pad 2: VCC -> +3.3V
- U1 pad 16: GND -> /NMOS
- U1 pad 2: GND -> /NMOS
- U1 pad 3: VCC -> +3.3V
- U1 pad 9: GND -> /NMOS
- U2 pad 1: VCC -> +3.3V
- U2 pad 3: /RST -> /BTN2
- U2 pad 5: /BTN2 -> /RST
Routing:
- net +3.3V: track 0.00 -> 100.8 mm
- net /STRAP: track 0.00 -> 51.4 mm, vias 0 -> 1
- net /NMOS: track 0.00 -> 50.9 mm
- net /BTN1: track 0.00 -> 41.0 mm, vias 0 -> 1
- net /UPDI: track 0.00 -> 33.1 mm, vias 0 -> 1
- net /BTN2: track 0.00 -> 29.1 mm, vias 0 -> 2
- net /RST: track 0.00 -> 25.6 mm, vias 0 -> 2
- net /DIO0: track 0.00 -> 22.1 mm, vias 0 -> 2
- net /CS: track 0.00 -> 13.0 mm
- net /LED2: track 0.00 -> 9.66 mm
- net /LED1: track 0.00 -> 7.75 mm
- net /MOSI: track 0.00 -> 6.61 mm
- net Net-(U1-ANT/NC): track 0.00 -> 6.35 mm
- net /MISO: track 0.00 -> 5.28 mm
- net /SCK: track 0.00 -> 3.90 mm
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- added copper zone on B.Cu, net GND
- added copper zone on F.Cu, net GND
Other:
- board size 30 x 70 mm -> 30 x 68.9 mm
- board text added: "ATtiny1624 LoRa Remote"
- board text removed: "3.3V"
- board text removed: "ATtiny85 LoRa Remote"
- board text removed: "GND"

Commit message: done
Parts:
- added REF**: SolderWirePad_1x01_SMD_1x2mm, Connector_Wire:SolderWirePad_1x01_SMD_1x2mm, F.Cu at (109.0, 85.1)
- added REF**: SolderWirePad_1x01_SMD_1x2mm, Connector_Wire:SolderWirePad_1x01_SMD_1x2mm, F.Cu at (116.6, 85.1)
- added REF**: SolderWirePad_1x01_SMD_1x2mm, Connector_Wire:SolderWirePad_1x01_SMD_1x2mm, B.Cu at (99.6, 46.5)
- added REF**: SolderWirePad_1x01_SMD_1x2mm, Connector_Wire:SolderWirePad_1x01_SMD_1x2mm, B.Cu at (99.6, 56.6)
- added REF**: SolderWirePad_1x01_SMD_1x2mm, Connector_Wire:SolderWirePad_1x01_SMD_1x2mm, B.Cu at (99.6, 51.5)
- added REF**: SolderWirePad_1x01_SMD_1x2mm, Connector_Wire:SolderWirePad_1x01_SMD_1x2mm, B.Cu at (99.7, 43.9)
- added REF**: SolderWirePad_1x01_SMD_1x2mm, Connector_Wire:SolderWirePad_1x01_SMD_1x2mm, B.Cu at (99.6, 54.1)
- added REF**: SolderWirePad_1x01_SMD_1x2mm, Connector_Wire:SolderWirePad_1x01_SMD_1x2mm, B.Cu at (99.6, 49.0)
- BT1: moved to B.Cu
- G***: moved to F.Cu
- moved G*** 7.27 mm to (115.1, 96.2), turned to 0 degrees
Routing:
- net /CS: track 13.0 -> 34.5 mm, vias 0 -> 1
- net /SCK: track 3.90 -> 24.9 mm, vias 0 -> 1
- net /MISO: track 5.28 -> 26.0 mm, vias 0 -> 1
- net /MOSI: track 6.61 -> 27.2 mm, vias 0 -> 1
- net /RST: track 25.6 -> 34.7 mm
- net +3.3V: track 100.8 -> 106.6 mm
- net /DIO0: track 22.1 -> 27.9 mm
- net GND: track 1.02 -> 1.70 mm, vias 23 -> 27
Other:
- outline, holes or cut-outs redrawn
- board text added: "+"
- board text added: "-"
- board text added: "CS"
- board text added: "DIO0"
- board text added: "MISO"
- board text added: "MOSI"
- board text added: "RST"
- board text added: "RX"
- board text added: "SCK"
- board text added: "STR"
- board text added: "TX"
- board text added: "UART0"
- board text added: "UPDI"
- board text removed: "PB5"
